File: sound-multi-board-hw-v1/sound-multi-board-hw-v1.kicad_pcb (KiCad board)
At the start: 2 copper layers, 100 x 100 mm, 37 parts, among them J1 USB_C_Receptacle_USB2.0_16P, J11 SWD, U1 NAU88C22, U10 STM32F405RGTx, U2 ESP32-WROOM-32, U3 USB3300-EZK, U4 STM32F407VGTx, Y1 12MHz 12pF, Y2 RTC 12.5pF

Commit message: choose between lqfp100 and 144
Parts:
- added U5: W9825G6KH-6, Package_SO:TSOP-II-54_22.2x10.16mm_P0.8mm, F.Cu at (206.2, 60.6)
- added U6: STM32F469VITx, Package_QFP:LQFP-100_14x14mm_P0.5mm, F.Cu at (156.3, 59.0)
- U4: value STM32F407VGTx -> STM32F479ZITx; footprint Package_QFP:LQFP-100_14x14mm_P0.5mm -> Package_QFP:LQFP-144_20x20mm_P0.5mm
- moved U4 0.67 mm to (181.3, 59.8)
Connections:
- U4 pad 10: Net-(U4-VSS-Pad10) -> unconnected-(U4-PF1-Pad10)
- U4 pad 15: unconnected-(U4-PC0-Pad15) -> Net-(U4-VSS-Pad109)
- U4 pad 27: Net-(U4-VSS-Pad10) -> unconnected-(U4-VREF+-Pad27)
- U4 pad 33: unconnected-(U4-PC4-Pad33) -> Net-(U4-VSS-Pad109)
- U4 pad 55: unconnected-(U4-PD8-Pad55) -> Net-(U4-VSS-Pad109)
- U4 pad 74: Net-(U4-VSS-Pad10) -> unconnected-(U4-PD11-Pad74)
- U4 pad 76: unconnected-(U4-PA14-Pad76) -> Net-(U4-VSS-Pad109)
- U4 pad 99: Net-(U4-VSS-Pad10) -> unconnected-(U4-PC7-Pad99)
